Commit message: meshes

File: public/cad/gpr-20241204.urdf (robot description, URDF)
Before this commit: robot gpr-20241204, 22 links, 21 joints
Links:
- added link arm-actuator, mass 0.4; collision mesh filename=meshes/arm-actuator.stl; visual mesh filename=meshes/arm-actuator.stl
- added link arm-actuator_2, mass 0.4; collision mesh filename=meshes/arm-actuator_2.stl; visual mesh filename=meshes/arm-actuator_2.stl
- added link arm-stopper-2.stp, mass 0.075787127; collision mesh filename=meshes/arm-stopper-2.stp.stl; visual mesh filename=meshes/arm-stopper-2.stp.stl
- added link arm-stopper-2.stp_2, mass 0.075787053; collision mesh filename=meshes/arm-stopper-2.stp_2.stl; visual mesh filename=meshes/arm-stopper-2.stp_2.stl
- added link arm2_actuator, mass 0.4; collision mesh filename=meshes/arm2_actuator.stl; visual mesh filename=meshes/arm2_actuator.stl
- added link arm2_actuator_2, mass 0.4; collision mesh filename=meshes/arm2_actuator_2.stl; visual mesh filename=meshes/arm2_actuator_2.stl
- added link arm3_actuator, mass 0.4; collision mesh filename=meshes/arm3_actuator.stl; visual mesh filename=meshes/arm3_actuator.stl
- added link arm3_actuator2, mass 0.4; collision mesh filename=meshes/arm3_actuator2.stl; visual mesh filename=meshes/arm3_actuator2.stl
- added link back_shell, mass 0.24321991; collision mesh filename=meshes/back_shell.stl; visual mesh filename=meshes/back_shell.stl
- added link body1-part_10, mass 0.5; collision mesh filename=meshes/body1-part_10.stl; visual mesh filename=meshes/body1-part_10.stl
- added link body1-part_11, mass 0.046132725; collision mesh filename=meshes/body1-part_11.stl; visual mesh filename=meshes/body1-part_11.stl
- added link body1-part_12, mass 0.55223125; collision mesh filename=meshes/body1-part_12.stl; visual mesh filename=meshes/body1-part_12.stl
- added link body1-part_13, mass 0.2184791; collision mesh filename=meshes/body1-part_13.stl; visual mesh filename=meshes/body1-part_13.stl
- added link body1-part_14, mass 0.15852082; collision mesh filename=meshes/body1-part_14.stl; visual mesh filename=meshes/body1-part_14.stl
- added link body1-part_15, mass 0.13419396; collision mesh filename=meshes/body1-part_15.stl; visual mesh filename=meshes/body1-part_15.stl
- added link body1-part_16, mass 0.9; collision mesh filename=meshes/body1-part_16.stl; visual mesh filename=meshes/body1-part_16.stl
- added link body1-part_17, mass 0.9; collision mesh filename=meshes/body1-part_17.stl; visual mesh filename=meshes/body1-part_17.stl
- added link body1-part_18, mass 2.65; collision mesh filename=meshes/body1-part_18.stl; visual mesh filename=meshes/body1-part_18.stl
- added link body1-part_19, mass 0.19664803; collision mesh filename=meshes/body1-part_19.stl; visual mesh filename=meshes/body1-part_19.stl
- added link body1-part_2, mass 0.9; collision mesh filename=meshes/body1-part_2.stl; visual mesh filename=meshes/body1-part_2.stl
- added link body1-part_20, mass 0.17091898; collision mesh filename=meshes/body1-part_20.stl; visual mesh filename=meshes/body1-part_20.stl
- added link body1-part_21, mass 0.067658274; collision mesh filename=meshes/body1-part_21.stl; visual mesh filename=meshes/body1-part_21.stl
- added link body1-part_22, mass 0.067658274; collision mesh filename=meshes/body1-part_22.stl; visual mesh filename=meshes/body1-part_22.stl
- added link body1-part_23, mass 0.17646959; collision mesh filename=meshes/body1-part_23.stl; visual mesh filename=meshes/body1-part_23.stl
- added link body1-part_3, mass 0.9; collision mesh filename=meshes/body1-part_3.stl; visual mesh filename=meshes/body1-part_3.stl
- added link body1-part_4, mass 0.58787898; collision mesh filename=meshes/body1-part_4.stl; visual mesh filename=meshes/body1-part_4.stl
- added link body1-part_5, mass 0.68030096; collision mesh filename=meshes/body1-part_5.stl; visual mesh filename=meshes/body1-part_5.stl
- added link body1-part_6, mass 0.075924533; collision mesh filename=meshes/body1-part_6.stl; visual mesh filename=meshes/body1-part_6.stl
- added link body1-part_7, mass 0.075924533; collision mesh filename=meshes/body1-part_7.stl; visual mesh filename=meshes/body1-part_7.stl
- added link body1-part_8, mass 0.021354804; collision mesh filename=meshes/body1-part_8.stl; visual mesh filename=meshes/body1-part_8.stl
- added link body1-part_9, mass 0.021354804; collision mesh filename=meshes/body1-part_9.stl; visual mesh filename=meshes/body1-part_9.stl
- added link foot2, mass 0.23284596; collision mesh filename=meshes/foot2.stl; visual mesh filename=meshes/foot2.stl
- added link foot4, mass 0.23284597; collision mesh filename=meshes/foot4.stl; visual mesh filename=meshes/foot4.stl
- added link front_shell, mass 0.44765499; collision mesh filename=meshes/front_shell.stl; visual mesh filename=meshes/front_shell.stl
- added link hand_actuator, mass 0.31; collision mesh filename=meshes/hand_actuator.stl; visual mesh filename=meshes/hand_actuator.stl
- added link hand_actuator_2, mass 0.31; collision mesh filename=meshes/hand_actuator_2.stl; visual mesh filename=meshes/hand_actuator_2.stl
- added link hand_part, mass 0.022065392; collision mesh filename=meshes/hand_part.stl; visual mesh filename=meshes/hand_part.stl
- added link hand_part2, mass 0.022065392; collision mesh filename=meshes/hand_part2.stl; visual mesh filename=meshes/hand_part2.stl
- added link hand_part2_2, mass 0.022065392; collision mesh filename=meshes/hand_part2_2.stl; visual mesh filename=meshes/hand_part2_2.stl
- added link hand_part_2, mass 0.022065392; collision mesh filename=meshes/hand_part_2.stl; visual mesh filename=meshes/hand_part_2.stl
- added link hand_shell2, mass 0.03852471; collision mesh filename=meshes/hand_shell2.stl; visual mesh filename=meshes/hand_shell2.stl
- added link hand_shell2_2, mass 0.03852471; collision mesh filename=meshes/hand_shell2_2.stl; visual mesh filename=meshes/hand_shell2_2.stl
- added link hand_umi, mass 0.064227671; collision mesh filename=meshes/hand_umi.stl; visual mesh filename=meshes/hand_umi.stl
- added link hand_umi2, mass 0.064227671; collision mesh filename=meshes/hand_umi2.stl; visual mesh filename=meshes/hand_umi2.stl
- added link hand_umi2_2, mass 0.064227671; collision mesh filename=meshes/hand_umi2_2.stl; visual mesh filename=meshes/hand_umi2_2.stl
- added link hand_umi_2, mass 0.064227671; collision mesh filename=meshes/hand_umi_2.stl; visual mesh filename=meshes/hand_umi_2.stl
- added link leg-stopper-2, mass 0.096079192; collision mesh filename=meshes/leg-stopper-2.stl; visual mesh filename=meshes/leg-stopper-2.stl
- added link leg-stopper-2_2, mass 0.096079242; collision mesh filename=meshes/leg-stopper-2_2.stl; visual mesh filename=meshes/leg-stopper-2_2.stl
- added link leg0_actuator, mass 0.9; collision mesh filename=meshes/leg0_actuator.stl; visual mesh filename=meshes/leg0_actuator.stl
- added link leg0_actuator_2, mass 0.9; collision mesh filename=meshes/leg0_actuator_2.stl; visual mesh filename=meshes/leg0_actuator_2.stl
- added link leg0_bearing, mass 0.053266787; collision mesh filename=meshes/leg0_bearing.stl; visual mesh filename=meshes/leg0_bearing.stl
- added link leg0_bearing_2, mass 0.053266787; collision mesh filename=meshes/leg0_bearing_2.stl; visual mesh filename=meshes/leg0_bearing_2.stl
- added link leg1_actuator, mass 0.9; collision mesh filename=meshes/leg1_actuator.stl; visual mesh filename=meshes/leg1_actuator.stl
- added link leg1_actuator2, mass 0.9; collision mesh filename=meshes/leg1_actuator2.stl; visual mesh filename=meshes/leg1_actuator2.stl
- added link leg2_actuator, mass 1.5; collision mesh filename=meshes/leg2_actuator.stl; visual mesh filename=meshes/leg2_actuator.stl
- added link leg2_actuator_2, mass 1.5; collision mesh filename=meshes/leg2_actuator_2.stl; visual mesh filename=meshes/leg2_actuator_2.stl
- added link leg2_bearing, mass 0.053266787; collision mesh filename=meshes/leg2_bearing.stl; visual mesh filename=meshes/leg2_bearing.stl
- added link leg2_bearing_2, mass 0.053266787; collision mesh filename=meshes/leg2_bearing_2.stl; visual mesh filename=meshes/leg2_bearing_2.stl
- added link leg3_actuator, mass 0.4; collision mesh filename=meshes/leg3_actuator.stl; visual mesh filename=meshes/leg3_actuator.stl
- added link leg3_actuator2, mass 0.4; collision mesh filename=meshes/leg3_actuator2.stl; visual mesh filename=meshes/leg3_actuator2.stl
- added link leg3_shell1, mass 0.56425494; collision mesh filename=meshes/leg3_shell1.stl; visual mesh filename=meshes/leg3_shell1.stl
- added link leg3_shell11, mass 0.56426179; collision mesh filename=meshes/leg3_shell11.stl; visual mesh filename=meshes/leg3_shell11.stl
- added link leg3_shell3, mass 0.14570047; collision mesh filename=meshes/leg3_shell3.stl; visual mesh filename=meshes/leg3_shell3.stl
- added link leg3_shell33, mass 0.14569982; collision mesh filename=meshes/leg3_shell33.stl; visual mesh filename=meshes/leg3_shell33.stl
- added link shoulder_3, mass 0.9; collision mesh filename=meshes/shoulder_3.stl; visual mesh filename=meshes/shoulder_3.stl
- added link shoulder_4, mass 0.6; collision mesh filename=meshes/shoulder_4.stl; visual mesh filename=meshes/shoulder_4.stl
- link arm1_top: mass 0.6485195170000001 -> 0.17273239
- link arm1_top_2: mass 0.648518913 -> 0.17273186
- link arm2_shell: mass 0.51101595 -> 0.11101595
- link arm2_shell_2: mass 0.51101595 -> 0.11101595
- link arm3_shell: mass 0.57887479 -> 0.17887479
- link arm3_shell2: mass 0.57887479 -> 0.17887479
- link body1-part: mass 11.923537116999999 -> 1.2310126
- link foot1: mass 0.54574734 -> 0.31290138
- link foot3: mass 0.5457471700000001 -> 0.3129012
- link hand_shell: mass 0.7933517460000001 -> 0.27224091
- link hand_shell_2: mass 0.7933517460000001 -> 0.27224091
- link leg0_shell: mass 1.3234480570000002 -> 0.37018127
- link leg0_shell_2: mass 1.3234480570000002 -> 0.37018127
- link leg1_shell: mass 1.360769512 -> 0.36469032
- link leg1_shell3: mass 1.360769362 -> 0.36469012
- link leg2_shell: mass 1.820922667 -> 0.26765588
- link leg2_shell_2: mass 1.820922667 -> 0.26765588
- link leg3_shell2: mass 1.179677561 -> 0.069722151
- link leg3_shell22: mass 1.179683991 -> 0.069722381
- link shoulder: mass 1.10769407 -> 0.20769407
- link shoulder_2: mass 0.80769287 -> 0.20769287
Joints:
- added joint Fastened_1: type fixed, parent body1-part_5, child body1-part_12, origin xyz=0.0375 -0.016 0.2911 rpy=3.1415927 0 3.1415927
- added joint Fastened_10: type fixed, parent body1-part_5, child body1-part_14, origin xyz=0.037 -0.0818 0.072175 rpy=0 0 3.1415927
- added joint Fastened_11: type fixed, parent body1-part_20, child body1-part_23, origin xyz=-1.307028e-05 0.098256596 -0.06658996 rpy=0 0 0
- added joint Fastened_12: type fixed, parent body1-part_14, child body1-part_20, origin xyz=0.097 -0.0116 0.048 rpy=-1.5707963 0 0
- added joint Fastened_13: type fixed, parent body1-part, child back_shell, origin xyz=0.039989396 0.07830385 -0.15700019 rpy=-1.5707963 0 1.5707963
- added joint Fastened_15: type fixed, parent body1-part, child front_shell, origin xyz=-0.040010604 0.07830385 -0.15700019 rpy=-1.5707963 0 1.5707963
- added joint Fastened_16: type fixed, parent body1-part, child body1-part_2, origin xyz=-1.0603759e-05 0.018089564 0.14549981 rpy=3.1415927 0 0
- added joint Fastened_17: type fixed, parent body1-part, child body1-part_3, origin xyz=-1.0603759e-05 0.018089564 -0.14550019 rpy=0 0 0
- added joint Fastened_18: type fixed, parent body1-part_3, child body1-part_7, origin xyz=0 0 -0.0395 rpy=0 0 0
- added joint Fastened_19: type fixed, parent body1-part_2, child body1-part_6, origin xyz=0 0 -0.0395 rpy=0 0 0
- added joint Fastened_1_10: type fixed, parent leg2_shell, child leg2_actuator, origin xyz=0 0.013 -0.1425 rpy=-1.5707963 0 0
- added joint Fastened_1_11: type fixed, parent leg2_shell_2, child leg2_actuator_2, origin xyz=0 0.013 -0.1425 rpy=-1.5707963 0 0
- added joint Fastened_1_12: type fixed, parent hand_shell, child hand_actuator, origin xyz=0 0 -0.062 rpy=3.1415927 0 0
- added joint Fastened_1_13: type fixed, parent hand_shell_2, child hand_actuator_2, origin xyz=0 0 -0.062 rpy=3.1415927 0 0
- added joint Fastened_1_14: type fixed, parent leg3_shell22, child leg3_shell11, origin xyz=-0.029 -0.068 0.0222 rpy=0 0 3.1415927
- added joint Fastened_1_15: type fixed, parent foot3, child foot4, origin xyz=0.11 -0.015 -0.0025 rpy=-1.5707963 0 0
- added joint Fastened_1_2: type fixed, parent shoulder_2, child shoulder_4, origin xyz=0.020011964 -5.6278452e-05 -0.0675 rpy=-1.5707963 0 -1.5707963
- added joint Fastened_1_3: type fixed, parent arm1_top_2, child arm-actuator_2, origin xyz=-0.108 0 0.0225 rpy=0 1.5707963 0
- added joint Fastened_1_4: type fixed, parent leg0_shell, child leg0_actuator, origin xyz=-0.0301 0 -0.0695 rpy=-1.5707963 0 1.5707963
- added joint Fastened_1_5: type fixed, parent leg0_shell_2, child leg0_actuator_2, origin xyz=-0.0301 0 -0.0695 rpy=-1.5707963 0 1.5707963
- added joint Fastened_1_6: type fixed, parent arm2_shell, child arm2_actuator, origin xyz=-0.0175 0 -0.098 rpy=0 -1.5707963 0
- added joint Fastened_1_7: type fixed, parent arm2_shell_2, child arm2_actuator_2, origin xyz=0.0175 0 0.0975 rpy=0 1.5707963 0
- added joint Fastened_1_8: type fixed, parent leg1_shell3, child leg1_actuator2, origin xyz=-0.0999 -0.00011981393 0.0275 rpy=0 1.5707963 0
- added joint Fastened_1_9: type fixed, parent arm3_shell2, child arm3_actuator2, origin xyz=-0.15 0 0.0215 rpy=3.1415927 -1.5707963 0
- added joint Fastened_2: type fixed, parent shoulder, child shoulder_3, origin xyz=0.020011964 5.6278452e-05 -0.0675 rpy=1.5707963 0 1.5707963
- added joint Fastened_20: type fixed, parent body1-part, child body1-part_4, origin xyz=-0.024510604 0.092089564 -0.050000186 rpy=-1.5707963 0 -3.1415927
- added joint Fastened_21: type fixed, parent body1-part_4, child body1-part_8, origin xyz=0.0067 -0.118 -0.0145 rpy=0 1.5707963 0
- added joint Fastened_22: type fixed, parent body1-part_4, child body1-part_9, origin xyz=0.0067 0.018 -0.0145 rpy=0 1.5707963 0
- added joint Fastened_23: type fixed, parent body1-part_4, child body1-part_10, origin xyz=-0.011681946 -0.05 -0.15525297 rpy=-1.5707963 0 0
- added joint Fastened_24: type fixed, parent body1-part_10, child body1-part_15, origin xyz=0.026228088 -0.096917942 0 rpy=0 0 0
- added joint Fastened_25: type fixed, parent body1-part_4, child body1-part_11, origin xyz=-0.0096448259 -0.049375 -0.12181656 rpy=-1.5707963 0 0
- added joint Fastened_2_10: type fixed, parent hand_shell, child hand_shell2, origin xyz=0 -0.029727738 -0.107 rpy=3.1415927 -1.5707963 0
- added joint Fastened_2_11: type fixed, parent hand_shell_2, child hand_shell2_2, origin xyz=0 -0.029727738 -0.107 rpy=3.1415927 -1.5707963 0
- added joint Fastened_2_12: type fixed, parent leg3_shell11, child leg3_actuator2, origin xyz=-0.029 0.042 0.0121 rpy=0 0 0
- added joint Fastened_2_13: type fixed, parent foot1, child foot2, origin xyz=0.125 -0.015 0.0015 rpy=-1.5707963 0 0
- added joint Fastened_2_2: type fixed, parent body1-part_12, child body1-part_16, origin xyz=0.0375 0.0647 -0.011 rpy=-1.5707963 0 0
- added joint Fastened_2_3: type fixed, parent arm1_top, child arm-actuator, origin xyz=-0.108 0 -0.0235 rpy=3.1415927 -1.5707963 0
- added joint Fastened_2_4: type fixed, parent leg0_shell, child leg0_bearing, origin xyz=-0.0346 0 -0.0695 rpy=1.5707963 0 1.5707963
- added joint Fastened_2_5: type fixed, parent leg0_shell_2, child leg0_bearing_2, origin xyz=-0.0346 0 -0.0695 rpy=1.5707963 0 1.5707963
- added joint Fastened_2_6: type fixed, parent leg1_shell, child leg1_actuator, origin xyz=-0.0999 0.00011981393 0.0275 rpy=0 1.5707963 0
- added joint Fastened_2_7: type fixed, parent arm3_shell, child arm3_actuator, origin xyz=-0.15 0 0.0215 rpy=3.1415927 -1.5707963 0
- added joint Fastened_2_8: type fixed, parent leg2_shell, child leg2_bearing, origin xyz=0 0.0307 -0.1425 rpy=1.5707963 0 0
- added joint Fastened_2_9: type fixed, parent leg2_shell_2, child leg2_bearing_2, origin xyz=0 0.0307 -0.1425 rpy=1.5707963 0 0
- added joint Fastened_3: type fixed, parent body1-part_12, child body1-part_17, origin xyz=0.0375 -0.0332 -0.011 rpy=-1.5707963 0 0
- added joint Fastened_3_2: type fixed, parent arm-actuator_2, child arm-stopper-2.stp_2, origin xyz=0 0 -0.028 rpy=0 0 1.5707963
- added joint Fastened_3_3: type fixed, parent leg1_actuator2, child leg-stopper-2_2, origin xyz=0 0 -0.0541 rpy=0 0 0
- added joint Fastened_3_4: type fixed, parent hand_shell2, child hand_part2, origin xyz=-0.0010182322 -0.042356503 -0.0545 rpy=3.1415927 0 0
- added joint Fastened_3_5: type fixed, parent hand_shell2_2, child hand_part2_2, origin xyz=-0.0010182322 -0.042356503 -0.0545 rpy=3.1415927 0 0
- added joint Fastened_3_6: type fixed, parent leg3_shell1, child leg3_actuator, origin xyz=-0.029 -0.042 0.0121 rpy=0 0 0
- added joint Fastened_4: type fixed, parent body1-part_16, child body1-part_21, origin xyz=0 0 0.039 rpy=3.1415927 0 0
- added joint Fastened_4_2: type fixed, parent arm-actuator, child arm-stopper-2.stp, origin xyz=0 0 -0.028 rpy=0 0 -1.5707963
- added joint Fastened_4_3: type fixed, parent leg1_actuator, child leg-stopper-2, origin xyz=0 0 -0.0566 rpy=0 0 0
- added joint Fastened_4_4: type fixed, parent leg3_shell11, child leg3_shell33, origin xyz=-0.029 0.042 0.047 rpy=3.1415927 0 0
- added joint Fastened_4_5: type fixed, parent hand_part, child hand_umi, origin xyz=-0.05 0.0125 0.0125 rpy=0 0 0
- added joint Fastened_4_6: type fixed, parent hand_part_2, child hand_umi_2, origin xyz=-0.05 0.0125 0.0125 rpy=0 0 0
- added joint Fastened_5: type fixed, parent body1-part_17, child body1-part_22, origin xyz=0 0 -0.039 rpy=0 0 0
- added joint Fastened_5_2: type fixed, parent hand_shell2, child hand_part, origin xyz=-0.0010182322 -0.017663497 0.0545 rpy=3.1415927 0 0
- added joint Fastened_5_3: type fixed, parent hand_shell2_2, child hand_part_2, origin xyz=-0.0010182322 -0.017663497 0.0545 rpy=3.1415927 0 0
- added joint Fastened_5_4: type fixed, parent leg3_shell1, child leg3_shell3, origin xyz=-0.029 -0.042 0.047 rpy=3.1415927 0 0
- added joint Fastened_6: type fixed, parent body1-part_13, child body1-part_18, origin xyz=0.001 -0.10185 0 rpy=-1.5707963 0 -1.5707963
- added joint Fastened_6_2: type fixed, parent leg3_shell2, child leg3_shell1, origin xyz=0.029 -0.068 0.0222 rpy=0 0 0
- added joint Fastened_6_3: type fixed, parent hand_part2, child hand_umi2, origin xyz=-0.05 -0.0125 -0.0125 rpy=3.1415927 0 0
- added joint Fastened_6_4: type fixed, parent hand_part2_2, child hand_umi2_2, origin xyz=-0.05 -0.0125 -0.0125 rpy=3.1415927 0 0
- added joint Fastened_7: type fixed, parent body1-part_13, child body1-part_19, origin xyz=-0.036 -0.165 -0.0725 rpy=-1.5707963 0 -1.5707963
- added joint Fastened_8: type fixed, parent body1-part, child body1-part_5, origin xyz=-1.0603691e-05 -0.12991044 0 rpy=1.5707963 0 0
- added joint Fastened_9: type fixed, parent body1-part_5, child body1-part_13, origin xyz=-0.035 0 0.23695 rpy=1.5707963 0 3.1415927
- joint L_ankle: origin xyz=0.0 -0.30000000004641003 0.07019999118206069 rpy=9.282041357749903e-08 0.0 0.0 -> xyz=0 0.19 -0.001 rpy=3.1415927 0 0; parent leg3_shell2 -> leg3_shell3
- joint L_elbow: child arm3_shell2 -> arm3_shell; limit lower=-2.0943951 upper=2.0943951 effort=80 velocity=5 -> lower=0 upper=2.7925268 effort=80 velocity=5; origin xyz=2.2775662092411332e-10 0.026000000000000002 0.0975 rpy=1.5707963999999996 1.5707963000000005 0.0 -> xyz=0 0 0.0085 rpy=3.1415927 0 0; parent arm2_shell_2 -> arm2_actuator
- joint L_hip_x: origin xyz=0.02649999999999997 -1.5165911463888016e-09 -0.06950000151659115 rpy=-1.5707963 0.0 1.5707963 -> xyz=0 0 -0.0566 rpy=0 0 0; parent leg0_shell -> leg0_actuator
- joint L_hip_y: origin xyz=-1.0608503738424868e-05 -0.43201043179234816 0.08770000686486731 rpy=-3.1415925071795874 4.641020678874952e-08 -3.1415926535897913 -> xyz=0 0 0.039 rpy=3.1415927 0 0; parent body1-part -> body1-part_16
- joint L_hip_z: origin xyz=-0.15649999999999997 0.00011981393 0.027499998483408852 rpy=-0.0 1.5707963 0.0 -> xyz=0 0 -0.0566 rpy=0 0 0; parent leg1_shell -> leg1_actuator
- joint L_knee: origin xyz=0.0 0.0342 -0.14250000009378214 rpy=1.5707963000000003 0.0 0.0 -> xyz=0 0 -0.0035 rpy=0 0 0; parent leg2_shell -> leg2_bearing
- joint L_shoulder_x: origin xyz=0.022511964 5.627838501275855e-05 -0.06749999993301277 rpy=1.5707963 0.0 1.5707963 -> xyz=0 0 0.0025 rpy=0 0 0; parent shoulder -> shoulder_3
- joint L_shoulder_y: origin xyz=-1.0603759e-05 0.018089562050771318 0.18749980999999996 rpy=3.1415926071795868 -2.220446049250313e-15 3.1415926071795868 -> xyz=0 0 -0.042 rpy=0 0 3.1415927; parent body1-part -> body1-part_2
- joint L_shoulder_z: origin xyz=-0.13949999999999996 -1.4619215099879723e-09 -0.02349999915596076 rpy=1.5707963535897933 -2.679489807810853e-08 1.5707963732051022 -> xyz=0 0 -0.0315 rpy=0 0 3.1415927; parent arm1_top -> arm-actuator
- joint L_wrist: origin xyz=-0.18149999999999997 -1.4619215099879723e-09 0.02150000084403924 rpy=-1.5707963535897926 -2.6794894969484062e-08 -1.5707962803846895 -> xyz=0 0 -0.0315 rpy=0 0 1.5707963; parent arm3_shell2 -> arm3_actuator2
- joint R_ankle: origin xyz=1.0767167917674625e-08 -0.2999999986541038 0.027200000000000002 rpy=-3.1415926071795868 2.220446049250313e-16 -3.1415926071795868 -> xyz=-0.029 0.232 0.005 rpy=3.1415927 0 0; parent leg3_shell22 -> leg3_shell11
- joint R_elbow: child arm3_shell -> arm3_shell2; limit lower=-2.0943951 upper=2.0943951 effort=80 velocity=5 -> lower=0 upper=2.7925268 effort=80 velocity=5; origin xyz=-0.026000000000000002 0.0 -0.09799999977224338 rpy=-3.1415926071795863 -1.5707963 0.0 -> xyz=0 0 0.0085 rpy=3.1415927 0 0; parent arm2_shell -> arm2_actuator_2
- joint R_hip_x: origin xyz=0.02649999999999997 -1.5165911463888016e-09 -0.06950000151659115 rpy=1.5707963 -4.641020634466031e-08 -1.5707963535897922 -> xyz=0 0 -0.0566 rpy=0 0 3.1415927; parent leg0_shell_2 -> leg0_actuator_2
- joint R_hip_y: origin xyz=-1.0600340183051227e-05 -0.4320104467591277 -0.08819999313513188 rpy=9.99999991702083e-08 4.641020678874952e-08 -3.1415926535897913 -> xyz=0 0 -0.039 rpy=0 0 0; parent body1-part -> body1-part_17
- joint R_hip_z: origin xyz=-0.15649999999999997 -0.00011981393 0.027499998483408852 rpy=-3.1415926535897922 -1.5707962732050302 0.0 -> xyz=0 0 -0.0566 rpy=0 0 3.1415927; parent leg1_shell3 -> leg1_actuator2
- joint R_knee: origin xyz=0.0 0.0342 -0.14250000009378214 rpy=1.5707963000000003 0.0 0.0 -> xyz=0 0 -0.0035 rpy=0 0 0; parent leg2_shell_2 -> leg2_bearing_2
- joint R_shoulder_x: origin xyz=0.022511964 -5.627838501275855e-05 -0.06749999993301277 rpy=1.5707963999999996 -2.220446049250313e-16 -1.5707963000000003 -> xyz=0 0 0.0025 rpy=3.1415927 0 0; parent shoulder_2 -> shoulder_4
- joint R_shoulder_y: origin xyz=-1.0603759e-05 0.018089564 -0.18750019 rpy=0.0 0.0 -3.1415926071795863 -> xyz=0 0 -0.042 rpy=0 0 3.1415927; parent body1-part -> body1-part_3
- joint R_shoulder_z: origin xyz=-0.13949999999999999 0.0 0.022499999155960758 rpy=-3.1415926071795863 1.5707963 0.0 -> xyz=0 0 -0.0315 rpy=3.1415927 0 0; parent arm1_top_2 -> arm-actuator_2
- joint R_wrist: origin xyz=-0.18149999999999997 -1.4619215099879723e-09 0.02150000084403924 rpy=-1.5707963535897926 -2.6794894969484062e-08 -1.5707962803846895 -> xyz=0 0 -0.0315 rpy=0 0 1.5707963; parent arm3_shell -> arm3_actuator
