Commit message: Updated URDF

File: public/cad/gpr-20241204.urdf (robot description, URDF)
Before this commit: robot gpr-20241204, 88 links, 87 joints
Links:
- removed link arm-actuator
- removed link arm-actuator_2
- removed link arm-stopper-2.stp
- removed link arm-stopper-2.stp_2
- removed link arm2_actuator
- removed link arm2_actuator_2
- removed link arm3_actuator
- removed link arm3_actuator2
- removed link back_shell
- removed link body1-part_10
- removed link body1-part_11
- removed link body1-part_12
- removed link body1-part_13
- removed link body1-part_14
- removed link body1-part_15
- removed link body1-part_16
- removed link body1-part_17
- removed link body1-part_18
- removed link body1-part_19
- removed link body1-part_2
- removed link body1-part_20
- removed link body1-part_21
- removed link body1-part_22
- removed link body1-part_23
- removed link body1-part_3
- removed link body1-part_4
- removed link body1-part_5
- removed link body1-part_6
- removed link body1-part_7
- removed link body1-part_8
- removed link body1-part_9
- removed link foot2
- removed link foot4
- removed link front_shell
- removed link hand_actuator
- removed link hand_actuator_2
- removed link hand_part
- removed link hand_part2
- removed link hand_part2_2
- removed link hand_part_2
- removed link hand_shell2
- removed link hand_shell2_2
- removed link hand_umi
- removed link hand_umi2
- removed link hand_umi2_2
- removed link hand_umi_2
- removed link leg-stopper-2
- removed link leg-stopper-2_2
- removed link leg0_actuator
- removed link leg0_actuator_2
- removed link leg0_bearing
- removed link leg0_bearing_2
- removed link leg1_actuator
- removed link leg1_actuator2
- removed link leg2_actuator
- removed link leg2_actuator_2
- removed link leg2_bearing
- removed link leg2_bearing_2
- removed link leg3_actuator
- removed link leg3_actuator2
- removed link leg3_shell1
- removed link leg3_shell11
- removed link leg3_shell3
- removed link leg3_shell33
- removed link shoulder_3
- removed link shoulder_4
- link arm1_top: mass 0.17273239 -> 1.104715355
- link arm1_top_2: mass 0.17273186 -> 1.1047097590000001
- link arm2_shell: mass 0.11101595 -> 0.8887392300000001
- link arm2_shell_2: mass 0.11101595 -> 0.88873928
- link arm3_shell: mass 0.17887479 -> 1.17434502
- link arm3_shell2: mass 0.17887479 -> 1.17434689
- link body1-part: mass 1.2310126 -> 11.923537116999999
- link foot1: mass 0.31290138 -> 0.54574734
- link foot3: mass 0.3129012 -> 0.5457471700000001
- link hand_shell: mass 0.27224091 -> 0.7933517460000001
- link hand_shell_2: mass 0.27224091 -> 0.7933517460000001
- link leg0_shell: mass 0.37018127 -> 1.3234480570000002
- link leg0_shell_2: mass 0.37018127 -> 1.3234480570000002
- link leg1_shell: mass 0.36469032 -> 2.3975352720000003
- link leg1_shell3: mass 0.36469012 -> 2.3975351220000003
- link leg2_shell: mass 0.26765588 -> 2.3673054970000003
- link leg2_shell_2: mass 0.26765588 -> 2.367304667
- link leg3_shell2: mass 0.069722151 -> 1.7593333310000001
- link leg3_shell22: mass 0.069722381 -> 1.7593397609999997
- link shoulder: mass 0.20769407 -> 1.2849791
- link shoulder_2: mass 0.20769287 -> 0.98497785
Joints:
- removed joint Fastened_1
- removed joint Fastened_10
- removed joint Fastened_11
- removed joint Fastened_12
- removed joint Fastened_13
- removed joint Fastened_15
- removed joint Fastened_16
- removed joint Fastened_17
- removed joint Fastened_18
- removed joint Fastened_19
- removed joint Fastened_1_10
- removed joint Fastened_1_11
- removed joint Fastened_1_12
- removed joint Fastened_1_13
- removed joint Fastened_1_14
- removed joint Fastened_1_15
- removed joint Fastened_1_2
- removed joint Fastened_1_3
- removed joint Fastened_1_4
- removed joint Fastened_1_5
- removed joint Fastened_1_6
- removed joint Fastened_1_7
- removed joint Fastened_1_8
- removed joint Fastened_1_9
- removed joint Fastened_2
- removed joint Fastened_20
- removed joint Fastened_21
- removed joint Fastened_22
- removed joint Fastened_23
- removed joint Fastened_24
- removed joint Fastened_25
- removed joint Fastened_2_10
- removed joint Fastened_2_11
- removed joint Fastened_2_12
- removed joint Fastened_2_13
- removed joint Fastened_2_2
- removed joint Fastened_2_3
- removed joint Fastened_2_4
- removed joint Fastened_2_5
- removed joint Fastened_2_6
- removed joint Fastened_2_7
- removed joint Fastened_2_8
- removed joint Fastened_2_9
- removed joint Fastened_3
- removed joint Fastened_3_2
- removed joint Fastened_3_3
- removed joint Fastened_3_4
- removed joint Fastened_3_5
- removed joint Fastened_3_6
- removed joint Fastened_4
- removed joint Fastened_4_2
- removed joint Fastened_4_3
- removed joint Fastened_4_4
- removed joint Fastened_4_5
- removed joint Fastened_4_6
- removed joint Fastened_5
- removed joint Fastened_5_2
- removed joint Fastened_5_3
- removed joint Fastened_5_4
- removed joint Fastened_6
- removed joint Fastened_6_2
- removed joint Fastened_6_3
- removed joint Fastened_6_4
- removed joint Fastened_7
- removed joint Fastened_8
- removed joint Fastened_9
- joint L_ankle: origin xyz=0 0.19 -0.001 rpy=3.1415927 0 0 -> xyz=0.0 -0.30000000004641003 0.07019999118206069 rpy=9.282041357749903e-08 0.0 0.0; parent leg3_shell3 -> leg3_shell2
- joint L_elbow: limit lower=0 upper=2.7925268 effort=80 velocity=5 -> lower=-2.5307274 upper=0 effort=80 velocity=5; origin xyz=0 0 0.0085 rpy=3.1415927 0 0 -> xyz=-0.026 0.0 -0.09799999977224338 rpy=-3.1415926071795863 -1.5707963 0.0; parent arm2_actuator -> arm2_shell
- joint L_hip_x: origin xyz=0 0 -0.0566 rpy=0 0 0 -> xyz=0.026499999999999965 -1.516591136963008e-09 -0.06950000151659115 rpy=-1.5707963 0.0 1.5707963; parent leg0_actuator -> leg0_shell
- joint L_hip_y: origin xyz=0 0 0.039 rpy=3.1415927 0 0 -> xyz=-1.0608503738440467e-05 -0.43201043179234816 0.08770000686486729 rpy=-3.1415925071795874 4.641020723283873e-08 -3.1415926535897913; parent body1-part_16 -> body1-part
- joint L_hip_z: origin xyz=0 0 -0.0566 rpy=0 0 0 -> xyz=-0.15649999999999997 0.00011981393 0.02749999848340886 rpy=-0.0 1.5707963 0.0; parent leg1_actuator -> leg1_shell
- joint L_knee: origin xyz=0 0 -0.0035 rpy=0 0 0 -> xyz=0.0 0.0342 -0.14250000009378214 rpy=1.5707963 0.0 0.0; parent leg2_bearing -> leg2_shell
- joint L_shoulder_x: origin xyz=0 0 0.0025 rpy=0 0 0 -> xyz=0.022511964 5.627838501275897e-05 -0.06749999993301277 rpy=1.5707963 2.220446049250313e-16 1.5707963; parent shoulder_3 -> shoulder
- joint L_shoulder_y: origin xyz=0 0 -0.042 rpy=0 0 3.1415927 -> xyz=-1.0603759e-05 0.018089562050771318 0.18749980999999996 rpy=3.1415926071795868 -2.220446049250313e-15 3.1415926071795868; parent body1-part_2 -> body1-part
- joint L_shoulder_z: origin xyz=0 0 -0.0315 rpy=0 0 3.1415927 -> xyz=-0.13949999999999996 -1.461921509987972e-09 -0.023499999155960766 rpy=-4.641020604450648e-08 1.5707962732050293 0.0; parent arm-actuator -> arm1_top
- joint L_wrist: origin xyz=0 0 -0.0315 rpy=0 0 1.5707963 -> xyz=-0.18149999999999994 -1.461921509987972e-09 0.021500000844039233 rpy=-1.5707963535897926 -2.6794894969484062e-08 -1.5707962803846893; parent arm3_actuator2 -> arm3_shell2
- joint R_ankle: origin xyz=-0.029 0.232 0.005 rpy=3.1415927 0 0 -> xyz=1.0767167917674625e-08 -0.29999999865410376 0.027200000000000002 rpy=-3.1415926071795868 0.0 -3.1415926071795868; parent leg3_shell11 -> leg3_shell22
- joint R_elbow: limit lower=0 upper=2.7925268 effort=80 velocity=5 -> lower=0 upper=2.5307274 effort=80 velocity=5; origin xyz=0 0 0.0085 rpy=3.1415927 0 0 -> xyz=0.026 0.0 0.09750000022775662 rpy=-3.1415926071795863 1.5707963 0.0; parent arm2_actuator_2 -> arm2_shell_2
- joint R_hip_x: origin xyz=0 0 -0.0566 rpy=0 0 3.1415927 -> xyz=0.026499999999999965 -1.516591136963008e-09 -0.06950000151659115 rpy=1.5707963 -4.641020678874952e-08 -1.5707963535897917; parent leg0_actuator_2 -> leg0_shell_2
- joint R_hip_y: origin xyz=0 0 -0.039 rpy=0 0 0 -> xyz=-1.0600340183049505e-05 -0.4320104467591277 -0.08819999313513191 rpy=9.99999991702083e-08 4.641020723283873e-08 -3.1415926535897913; parent body1-part_17 -> body1-part
- joint R_hip_z: origin xyz=0 0 -0.0566 rpy=0 0 3.1415927 -> xyz=-0.15649999999999997 -0.00011981393 0.02749999848340886 rpy=-3.1415926535897922 -1.5707962732050305 0.0; parent leg1_actuator2 -> leg1_shell3
- joint R_knee: origin xyz=0 0 -0.0035 rpy=0 0 0 -> xyz=0.0 0.0342 -0.14250000009378214 rpy=1.5707963 0.0 0.0; parent leg2_bearing_2 -> leg2_shell_2
- joint R_shoulder_x: origin xyz=0 0 0.0025 rpy=3.1415927 0 0 -> xyz=0.022511964 -5.627838501275897e-05 -0.06749999993301277 rpy=1.5707963999999996 2.220446049250313e-16 -1.5707963000000003; parent shoulder_4 -> shoulder_2
- joint R_shoulder_y: origin xyz=0 0 -0.042 rpy=0 0 3.1415927 -> xyz=-1.0603759e-05 0.018089564 -0.18750019 rpy=0.0 0.0 -3.1415926071795863; parent body1-part_3 -> body1-part
- joint R_shoulder_z: origin xyz=0 0 -0.0315 rpy=3.1415927 0 0 -> xyz=-0.13949999999999999 0.0 0.02249999915596076 rpy=-3.1415926071795863 1.5707963 0.0; parent arm-actuator_2 -> arm1_top_2
- joint R_wrist: origin xyz=0 0 -0.0315 rpy=0 0 1.5707963 -> xyz=-0.18149999999999994 -1.461921509987972e-09 0.021500000844039233 rpy=-1.5707963535897926 -2.6794894969484062e-08 -1.5707962803846893; parent arm3_actuator -> arm3_shell
